File: pcb/serialtap-r1p0/serialtap-r1p0.kicad_pcb (KiCad board)
At the start: 2 copper layers, 0 parts

Commit message: port: the service connector is 5-pin XA, not 4
Confirmed on the AS50QDFHRA, mated with a JST XARR-05V panel housing -
XA series, 2.5 mm pitch. The series assumption held; the pin count did
not.

The board carries a 5-pin header so the harness can be straight-through,
which is the least error-prone cable to build. Board-side candidates
recorded in SPDD 5.2; not pinned yet, because entry direction is a
mechanical call and the gender/mating relationship should be read off
the JST datasheet rather than a distributor summary.

The fifth pin connects to nothing - not the ESD array, not a GPIO -
until its function is captured. Strapping an unknown signal, possibly
not 5 V logic, to a net that matters is a worse failure than losing a
pin.

Also records the hand-drawn 40 x 25 mm outline, which verified that hand
edits to the .kicad_pcb survive ato build (SPDD 6's central claim, now
tested rather than assumed) and clears the DRC outline violation.

Co-Authored-By: Claude Opus 5 <noreply@anthropic.com>
Other:
- board outline added: 40 x 25 mm
Changed lines of the file:
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@@
 		)
 	)
+	(gr_rect
+		(start 100 100)
+		(end 140 125)
+		(stroke
+			(width 0.1)
+			(type default)
+		)
+		(fill no)
+		(layer "Edge.Cuts")
+	)
 )

Commit message: pcb: add the KiCad project file and the 4-layer stackup
atopile generates only a .kicad_pcb, and a default 2-layer one, so the
board could not be opened as a project and contradicted SPDD 8. Both
fixed by hand - the .kicad_pro and the stackup are hand-maintained
files, not build artifacts.

The project file carries the DRC values and net classes from
docs/layout-rules.md. Verified they are actually enforced, not merely
stored, by feeding kicad-cli a 0.05 mm track and confirming it was
rejected against the 0.127 mm minimum.

Four copper layers named per layout-rules.md. The dielectric heights are
the usual nominal figures for a 1.6 mm four-layer board and are marked
PROVISIONAL: layout-rules.md requires PCBWay's published stackup before
any trace geometry is computed, because the L1-L2 prepreg height sets
the USB pair dimensions.

Confirmed ato build preserves all of it - layers, stackup, outline and
the project file.

Co-Authored-By: Claude Opus 5 <noreply@anthropic.com>
Other:
- copper layers 2 -> 4
Changed lines of the file:
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@@
 	(layers
 		(0 "F.Cu" signal)
-		(31 "B.Cu" signal)
+		(1 "In1.Cu" power "GND (L2)")
+		(2 "In2.Cu" power "Rails (L3)")
+		(31 "B.Cu" power "GND (L4)")
 		(32 "B.Adhes" user "B.Adhesive")
 		(33 "F.Adhes" user "F.Adhesive")
@@
 			)
 			(layer "dielectric 1"
-				(type "core")
-				(thickness 1.51)
+				(type "prepreg")
+				(thickness 0.2104)
 				(material "FR4")
 				(epsilon_r 4.5)
+				(loss_tangent 0.02)
+			)
+			(layer "In1.Cu"
+				(type "copper")
+				(thickness 0.0175)
+			)
+			(layer "dielectric 2"
+				(type "core")
+				(thickness 1.065)
+				(material "FR4")
+				(epsilon_r 4.5)
+				(loss_tangent 0.02)
+			)
+			(layer "In2.Cu"
+				(type "copper")
+				(thickness 0.0175)
+			)
+			(layer "dielectric 3"
+				(type "prepreg")
+				(thickness 0.2104)
+				(material "FR4")
+				(epsilon_r 4.5)
