File: pcb/serialtap-r1p0.kicad_pcb (KiCad board)
At the start: 4 copper layers, 54 x 22 mm, 46 parts, among them J1 B05B-XASK-1-A, J2 USB4085-GF-A, SW1 SW_Push, SW2 SW_Push, U1 TPS2553DBV, U2 LM66200DRL, U3 TPS62162DSG, U4 TXU0204RUT, U5 TPD4E05U06DQA, U6 ESP32-C3-MINI-1

Commit message: Work the pre-release checklist, and sense VOS at the output capacitor
Checked from the board file: antenna keepout, L2 continuity, buck input loop,
switch node, TVS order, translator decoupling and tie-offs, test points,
silkscreen and DRC all pass, with measurements recorded in layout-rules.md.

The one failure was U3's VOS line, which tapped L1's output pad and ran along
the inductor body past the SW pad. Rerouted (by hand, in KiCad) to drop
through a via to L3 and come up at C6's pad — the topology of TI's layout
example, Figure 42 of the TPS62162 datasheet.

missing_courtyard is now a DRC error rather than ignored: every footprint
has one, and a future one without should not pass silently. Two stale
"antenna overhangs the outline" lines are marked superseded by the OEM
outline. DRC 0 violations, 0 unconnected, 0 parity.

Co-Authored-By: Claude Opus 5.5 <noreply@anthropic.com>
Routing:
- net V3V3: track 84.2 -> 86.1 mm, vias 7 -> 8
Changed lines of the file:
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@@
 	(segment
 		(start 135.4 118.25)
-		(end 135.4 120.9)
+		(end 135.4 119.3)
 		(width 0.3)
 		(layer "F.Cu")
@@
 	)
 	(segment
-		(start 139.59 120.9)
-		(end 139.59 120)
-		(width 0.3)
+		(start 143.1 120.5)
+		(end 143.1 119.675)
+		(width 0.5)
 		(layer "F.Cu")
 		(net "V3V3")
@@
 	)
 	(segment
-		(start 135.4 120.9)
-		(end 139.59 120.9)
-		(width 0.3)
-		(layer "F.Cu")
-		(net "V3V3")
-	)
-	(segment
 		(start 121.4 107.4)
 		(end 120.62 107.4)
@@
 	)
 	(via
+		(at 143.1 120.5)
+		(size 0.5)
+		(drill 0.25)
+		(layers "F.Cu" "B.Cu")
+		(net "V3V3")
+	)
+	(via
 		(at 112.03 120.9)
 		(size 0.5)
@@
 		(layer "In2.Cu")
 		(net "V3V3")
+	)
+	(segment
+		(start 135.4 120.5)
+		(end 143.1 120.5)
+		(width 0.5)
+		(layer "In2.Cu")
+		(net "V3V3")
